File: PCB/stor/stor.kicad_pcb (KiCad board)
At the start: 4 copper layers, 22 x 58.8 mm, 56 parts, among them J1 Conn_01x05_Socket, J2 Conn_01x04_Socket, SW1 TS1603-TZ38HBM, SW2 TS1603-TZ38HBM, U1 STM32H723VGT6, U3 USB3300-EZK-TR, U4 TPS62177DQCR, X1 25mhz, X2 32.768k, X3 24mhz

Commit message: Update stor.kicad_pcb
Parts:
- moved D1 0.09 mm to (123.2, 42.3)
Routing:
- net /PC11: track 39.4 -> 38.5 mm
- net /BOOT0: track 45.6 -> 46.3 mm
- net /VDD: track 51.6 -> 50.9 mm

Commit message: new usb
Parts:
- removed R2: 5.1k, easyeda2kicad:R0402
- C17: footprint easyeda2kicad:C0402 -> easyeda2kicad:C0603
- USB1: value GT-USB-8016A -> U-USBAR04P-M001; footprint easyeda2kicad:USB-TYPE-C-SMD_GT-USB-8016A -> easyeda2kicad:USB-SMD_KH-USB-AM-4P-CB
- moved C17 7.83 mm to (128.7, 46.1), turned to 180 degrees
- moved USB1 0.30 mm to (120.0, 37.9)
Connections:
- USB1 pad 1: GND -> /VBUS
- USB1 pad 2: GND -> /D-
- USB1 pad 3: GND -> /D+
Routing:
- net /PC8: track 42.2 -> 2.35 mm, vias 2 -> 0
- net /BOOT0: track 46.3 -> 11.7 mm, vias 3 -> 2
- net /PC9: track 35.8 -> 14.3 mm, vias 2 -> 1
- net GND: track 82.0 -> 68.5 mm, vias 59 -> 57
- net /CC1: track 9.52 -> 0.00 mm, vias 2 -> 0
- net /VBUS: track 41.4 -> 45.0 mm, vias 2 -> 5
- net /D-: track 19.0 -> 21.6 mm
- net /VDD: track 50.9 -> 52.4 mm
- net /PA7: track 8.43 -> 7.57 mm
- net /D+: track 17.9 -> 17.3 mm
- net /PB11: track 21.6 -> 21.0 mm
- net /PA6: track 8.04 -> 7.39 mm
Other:
- board size 22 x 58.8 mm -> 22 x 60.5 mm

Commit message: bom opt!!
Routing:
- net /PC8: track 2.35 -> 41.3 mm, vias 0 -> 2
- net /PC9: track 14.3 -> 39.5 mm, vias 1 -> 2
- net /BOOT0: track 11.7 -> 33.7 mm, vias 2 -> 4
- net GND: track 68.5 -> 73.3 mm
- net /PB11: track 21.0 -> 22.7 mm
- net /PB13: track 18.7 -> 20.4 mm
- net /PB12: track 19.9 -> 20.7 mm
- net /PC10: track 40.7 -> 41.3 mm

Commit message: Update stor.kicad_pcb
Routing:
- net GND: track 73.3 -> 71.9 mm, vias 57 -> 60
- net /D-: track 21.6 -> 20.8 mm
- net /VBUS: track 44.7 -> 44.0 mm, vias 5 -> 4
- net /PB11: track 22.7 -> 22.0 mm
- net /BOOT0: track 33.7 -> 33.0 mm
