File: PCB/stor/stor.kicad_pcb (KiCad board)
At the start: 4 copper layers, 22 x 60.5 mm, 55 parts, among them J1 Conn_01x05_Socket, J2 Conn_01x04_Socket, SW1 TS1603-TZ38HBM, SW2 TS1603-TZ38HBM, U1 STM32H723VGT6, U3 USB3300-EZK-TR, U4 TPS62177DQCR, X1 25mhz, X2 32.768k, X3 24mhz

Commit message: rbias placement
Parts:
- moved R5 19.1 mm to (111.8, 39.1), turned to 0 degrees
Routing:
- net Net-(U3-RBIAS): track 16.0 -> 8.22 mm
- net /D+: track 16.8 -> 17.7 mm
- net GND: track 71.9 -> 72.4 mm, vias 60 -> 57
Changed lines of the file:
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@@
 	(footprint "easyeda2kicad:R0402"
 		(layer "F.Cu")
-		(at 128.6 48.3 180)
+		(at 111.845 39.1)
 		(descr "200KΩ (2003) ±1%")
 		(property "Reference" "R5"
@@
 		)
 		(property "Manufacturer" "UNI-ROYAL"
-			(at 0 0 180)
+			(at 0 0 0)
 			(unlocked yes)
 			(layer "F.Fab")
@@
 		)
 		(property "MPN" "0402WGF1202TCE"
-			(at 0 0 180)
+			(at 0 0 0)
 			(unlocked yes)
 			(layer "F.Fab")
@@
 		(duplicate_pad_numbers_are_jumpers no)
 		(fp_line
-			(start 0.94 0.5)
-			(end 0.94 -0.5)
+			(start -0.94 -0.5)
+			(end -0.23 -0.5)
 			(stroke
 				(width 0.15)
@@
 		)
 		(fp_line
-			(start 0.94 -0.5)
-			(end 0.23 -0.5)
+			(start -0.94 0.5)
+			(end -0.94 -0.5)
 			(stroke
 				(width 0.15)
@@
 		)
 		(fp_line
-			(start 0.23 0.5)
-			(end 0.94 0.5)
+			(start -0.23 0.5)
+			(end -0.94 0.5)
 			(stroke
 				(width 0.15)
@@
 		)
 		(fp_line
-			(start -0.23 0.5)
-			(end -0.94 0.5)
+			(start 0.23 0.5)
+			(end 0.94 0.5)
 			(stroke
 				(width 0.15)
@@
 		)
 		(fp_line
-			(start -0.94 0.5)
-			(end -0.94 -0.5)
+			(start 0.94 -0.5)
+			(end 0.23 -0.5)
 			(stroke
 				(width 0.15)
@@
 		)
 		(fp_line
-			(start -0.94 -0.5)
-			(end -0.23 -0.5)
+			(start 0.94 0.5)
+			(end 0.94 -0.5)
 			(stroke
 				(width 0.15)
@@
 		)
 		(fp_line
-			(start 0.5 0.25)
-			(end -0.5 0.25)
+			(start -0.5 -0.25)
+			(end 0.5 -0.25)
 			(stroke
 				(width 0.05)
@@
 		)
 		(fp_line
-			(start 0.5 -0.25)
-			(end 0.5 0.25)
+			(start -0.5 0.25)
+			(end -0.5 -0.25)
 			(stroke
 				(width 0.05)
@@
 		)
 		(fp_line
-			(start -0.5 0.25)
-			(end -0.5 -0.25)
+			(start 0.5 -0.25)
+			(end 0.5 0.25)
 			(stroke
 				(width 0.05)
@@
 		)
 		(fp_line
-			(start -0.5 -0.25)
-			(end 0.5 -0.25)
+			(start 0.5 0.25)
+			(end -0.5 0.25)
 			(stroke
 				(width 0.05)
@@
 		)
 		(pad "1" smd rect
-			(at -0.43 0 180)
+			(at -0.43 0)
 			(size 0.566 0.54)
 			(layers "F.Cu" "F.Mask" "F.Paste")
@@
 		)
 		(pad "2" smd rect
-			(at 0.43 0 180)
+			(at 0.43 0)
 			(size 0.566 0.54)
 			(layers "F.Cu" "F.Mask" "F.Paste")
@@
 	)
 	(segment
+		(start 116.81 76.74)
+		(end 116.75 76.8)
+		(width 0.2)
+		(layer "F.Cu")
+		(net "GND")
+	)
+	(segment
 		(start 120.818874 42.838874)
 		(end 120.818874 41.978793)
@@
 	)
 	(segment
-		(start 117.530002 76.74)
-		(end 117.35 76.920002)
-		(width 0.2)
-		(layer "F.Cu")
-		(net "GND")
-	)
-	(segment
-		(start 117.88 76.74)
-		(end 117.530002 76.74)
+		(start 116.81 76.74)
+		(end 117.88 76.74)
 		(width 0.2)
 		(layer "F.Cu")
@@
 	)
 	(via
-		(at 117.35 76.920002)
-		(size 0.6)
-		(drill 0.3)
-		(layers "F.Cu" "B.Cu")
-		(net "GND")
-	)
-	(via
 		(at 120.01058 58.32982)
 		(size 0.6)
@@
 	)
 	(via
-		(at 110 85)
-		(size 0.6)
-		(drill 0.3)
-		(layers "F.Cu" "B.Cu")
-		(free yes)
-		(net "GND")
-	)
-	(via
 		(at 113.99 66.73)
 		(size 0.6)
@@
 	)
 	(via
-		(at 112.5 82.5)
-		(size 0.6)
-		(drill 0.3)
-		(layers "F.Cu" "B.Cu")
-		(free yes)
-		(net "GND")
-	)
-	(via
 		(at 120 85)
 		(size 0.6)
@@
 	)
 	(via
-		(at 111.15 38.8)
+		(at 116.75 76.8)
 		(size 0.6)
 		(drill 0.3)
 		(layers "F.Cu" "B.Cu")
-		(free yes)
 		(net "GND")
 	)
@@
 	)
 	(segment
+		(start 122.709071 40.862276)
+		(end 122.709071 38.552337)
+		(width 0.2032)
+		(layer "F.Cu")
+		(net "/D-")
+	)
+	(segment
 		(start 124.700929 42.012276)
 		(end 123.550929 40.862276)
@@
 	)
 	(segment
-		(start 122.709071 38.550074)
-		(end 122.709071 40.862276)
-		(width 0.2032)
-		(layer "F.Cu")
-		(net "/D-")
-	)
-	(segment
-		(start 119 38.2375)
-		(end 119.9875 37.25)
+		(start 122.709071 38.552337)
+		(end 121.406734 37.25)
 		(width 0.2032)
 		(layer "F.Cu")
@@
 	)
 	(segment
-		(start 121.408997 37.25)
-		(end 122.709071 38.550074)
+		(start 121.406734 37.25)
+		(end 119.9875 37.25)
 		(width 0.2032)
 		(layer "F.Cu")
@@
 	(segment
 		(start 119.9875 37.25)
-		(end 121.408997 37.25)
+		(end 119 38.2375)
 		(width 0.2032)
 		(layer "F.Cu")
@@
 	)
 	(segment
-		(start 121 38.9875)
-		(end 121 39.175)
+		(start 113.106089 42.156089)
+		(end 113.25 42.3)
 		(width 0.2032)
 		(layer "F.Cu")
@@
 	)
 	(segment
-		(start 113.106089 42.156089)
-		(end 113.25 42.3)
+		(start 113.106089 40.712109)
+		(end 113.106089 42.156089)
 		(width 0.2032)
 		(layer "F.Cu")
@@
 	)
 	(segment
-		(start 113.106089 40.712109)
-		(end 113.106089 42.156089)
+		(start 121.435281 41.730869)
+		(end 121.759071 42.054659)
 		(width 0.2032)
 		(layer "F.Cu")
@@
 	)
 	(segment
-		(start 121.318874 39.306374)
-		(end 121.318874 42.067527)
+		(start 121 39)
+		(end 121.435281 39.435281)
 		(width 0.2032)
 		(layer "F.Cu")
@@
 	)
 	(segment
-		(start 121.318874 42.067527)
+		(start 121.759071 42.054659)
 		(end 121.759071 42.507724)
 		(width 0.2032)
@@
 	)
 	(segment
+		(start 121.435281 39.435281)
+		(end 121.435281 41.730869)
+		(width 0.2032)
+		(layer "F.Cu")
+		(net "/D+")
+	)
+	(segment
+		(start 121.435281 39.422781)
+		(end 121 38.9875)
+		(width 0.2032)
+		(layer "F.Cu")
+		(net "/D+")
+	)
+	(segment
 		(start 113.343198 40.475)
 		(end 113.106089 40.712109)
@@
 	)
 	(segment
-		(start 128.17 47.63)
-		(end 128.18 47.62)
+		(start 112.275 39.1)
+		(end 112.275 39.2)
 		(width 0.2)
 		(layer "F.Cu")
@@
 	)
 	(segment
-		(start 128.17 48.3)
-		(end 128.17 47.63)
+		(start 112.275 39.2)
+		(end 111.575 39.9)
 		(width 0.2)
 		(layer "F.Cu")
@@
 	)
 	(via
-		(at 128.18 47.62)
+		(at 111.575 39.9)
 		(size 0.6)
 		(drill 0.3)
@@
 	)
 	(segment
-		(start 124.096857 45.073143)
-		(end 126.896857 47.873143)
+		(start 111.575 39.9)
+		(end 112.125 39.9)
 		(width 0.2)
 		(layer "B.Cu")
@@
 	)
 	(segment
-		(start 120.094107 42.044868)
-		(end 120.66 42.610761)
+		(start 112.125 39.9)
+		(end 114.390663 39.9)
 		(width 0.2)
 		(layer "B.Cu")
@@
 	)
 	(segment
-		(start 120.66 42.610761)
-		(end 120.66 44.46)
-		(width 0.2)
-		(layer "B.Cu")
-		(net "Net-(U3-RBIAS)")
-	)
-	(segment
-		(start 117.239973 42.74931)
-		(end 117.239973 42.455827)
-		(width 0.2)
-		(layer "B.Cu")
-		(net "Net-(U3-RBIAS)")
-	)
-	(segment
-		(start 127.926857 47.873143)
-		(end 128.18 47.62)
-		(width 0.2)
-		(layer "B.Cu")
-		(net "Net-(U3-RBIAS)")
-	)
-	(segment
-		(start 121.273143 45.073143)
-		(end 124.096857 45.073143)
-		(width 0.2)
-		(layer "B.Cu")
-		(net "Net-(U3-RBIAS)")
-	)
-	(segment
-		(start 117.650931 42.044868)
-		(end 120.094107 42.044868)
-		(width 0.2)
-		(layer "B.Cu")
-		(net "Net-(U3-RBIAS)")
-	)
-	(segment
-		(start 120.66 44.46)
-		(end 121.273143 45.073143)
-		(width 0.2)
-		(layer "B.Cu")
-		(net "Net-(U3-RBIAS)")
-	)
-	(segment
-		(start 126.896857 47.873143)
-		(end 127.926857 47.873143)
-		(width 0.2)
-		(layer "B.Cu")
-		(net "Net-(U3-RBIAS)")
-	)
-	(segment
-		(start 117.239973 42.455827)
-		(end 117.650931 42.044868)
+		(start 114.390663 39.9)
+		(end 117.239973 42.74931)
 		(width 0.2)
 		(layer "B.Cu")

Commit message: production 2!
Parts:
- added TP1: TestPoint, TestPoint:TestPoint_Pad_2.0x2.0mm, B.Cu at (128.0, 47.2)
- added TP2: TestPoint, TestPoint:TestPoint_Pad_2.0x2.0mm, B.Cu at (128.0, 52.2)
- added TP3: TestPoint, TestPoint:TestPoint_Pad_2.0x2.0mm, B.Cu at (128.0, 57.2)
Routing:
- net /VBUS: track 44.0 -> 48.9 mm
- net /VDD: track 52.4 -> 54.9 mm, vias 24 -> 25
- net GND: track 72.4 -> 73.3 mm
Other:
- board text added: "STM32H7 inside"
- board text added: "Sandisk Gaming"
- board text added: "TM"
- board text added: "USB2.0"
- board text added: "flash by"
- board text added: "闪迪高速游戏卡"
- board text removed: "STM32H723VGT6 inside"

Commit message: tt
Routing:
- net /VDD: track 54.9 -> 56.7 mm, vias 25 -> 24
- net GND: track 73.3 -> 74.7 mm
Changed lines of the file:
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@@
 	)
 	(segment
+		(start 120.74 78.66)
+		(end 120.74 79.65)
+		(width 0.2)
+		(layer "F.Cu")
+		(net "/VDD")
+	)
+	(segment
 		(start 125 64.1)
 		(end 125 65.1)
@@
 	)
 	(segment
+		(start 120.13 78.05)
+		(end 120.74 78.66)
+		(width 0.2)
+		(layer "F.Cu")
+		(net "/VDD")
+	)
+	(segment
 		(start 113.75 50)
 		(end 114.275997 50)
@@
 	)
 	(via
-		(at 120.74 79.65)
-		(size 0.6)
-		(drill 0.3)
-		(layers "F.Cu" "B.Cu")
-		(net "/VDD")
-	)
-	(via
 		(at 111.14 40.76)
 		(size 0.6)
@@
 	)
 	(segment
+		(start 118.54 79.65)
+		(end 118.54 80.35)
+		(width 0.2)
+		(layer "F.Cu")
+		(net "GND")
+	)
+	(segment
 		(start 128.25 49.77)
 		(end 128.25 50.16)
@@
 	)
 	(segment
+		(start 118.54 80.35)
+		(end 118.04 80.85)
+		(width 0.2)
+		(layer "F.Cu")
+		(net "GND")
+	)
+	(segment
 		(start 120.2 43.25)
 		(end 121.1 44.15)
@@
 	)
 	(via
-		(at 118.66962 79.77962)
-		(size 0.6)
-		(drill 0.3)
-		(layers "F.Cu" "B.Cu")
-		(net "GND")
-	)
-	(via
 		(at 128.84 45.400002)
 		(size 0.6)
@@
 	)
 	(via
+		(at 118.04 80.85)
+		(size 0.6)
+		(drill 0.3)
+		(layers "F.Cu" "B.Cu")
+		(net "GND")
+	)
+	(via
 		(at 120 90)
 		(size 0.6)
@@
 	)
 	(segment
-		(start 125.309925 72.785)
-		(end 125.925 72.169925)
+		(start 117.9 52.819239)
+		(end 117.145778 52.065017)
+		(width 0.2)
+		(layer "B.Cu")
+		(net "/PA9")
+	)
+	(segment
+		(start 117.9 54.024264)
+		(end 117.9 52.819239)
 		(width 0.2)
 		(layer "B.Cu")
@@
 	)
 	(segment
-		(start 122.088736 73.087)
-		(end 123.947264 73.087)
+		(start 125.134189 61.258453)
+		(end 117.9 54.024264)
 		(width 0.2)
 		(layer "B.Cu")
@@
 	)
 	(segment
-		(start 117.86962 77.306116)
-		(end 122.088736 73.087)
+		(start 117.86962 78.556877)
+		(end 117.86962 77.306116)
 		(width 0.2)
 		(layer "B.Cu")
@@
 	)
 	(segment
-		(start 125.134189 61.258453)
-		(end 117.9 54.024264)
+		(start 123.947264 73.087)
+		(end 124.249265 72.785)
 		(width 0.2)
 		(layer "B.Cu")
@@
 	)
 	(segment
-		(start 117.9 52.819239)
-		(end 117.145778 52.065017)
+		(start 117.28 79.6)
+		(end 117.28 79.146497)
 		(width 0.2)
 		(layer "B.Cu")
@@
 	)
 	(segment
-		(start 125.925 71.300075)
-		(end 125.134189 70.509264)
+		(start 117.86962 77.306116)
+		(end 122.088736 73.087)
 		(width 0.2)
 		(layer "B.Cu")
@@
 	)
 	(segment
-		(start 117.86962 79.01038)
-		(end 117.86962 77.306116)
+		(start 125.309925 72.785)
+		(end 125.925 72.169925)
 		(width 0.2)
 		(layer "B.Cu")
@@
 	)
 	(segment
-		(start 117.9 54.024264)
-		(end 117.9 52.819239)
+		(start 110.8 86.08)
+		(end 117.28 79.6)
 		(width 0.2)
 		(layer "B.Cu")
@@
 	)
 	(segment
-		(start 123.947264 73.087)
-		(end 124.249265 72.785)
+		(start 117.28 79.146497)
+		(end 117.86962 78.556877)
 		(width 0.2)
 		(layer "B.Cu")
@@
 	)
 	(segment
-		(start 110.8 86.08)
-		(end 117.86962 79.01038)
+		(start 125.925 71.300075)
+		(end 125.134189 70.509264)
+		(width 0.2)
+		(layer "B.Cu")
+		(net "/PA9")
+	)
+	(segment
+		(start 122.088736 73.087)
+		(end 123.947264 73.087)
 		(width 0.2)
 		(layer "B.Cu")
@@
 	)
 	(segment
-		(start 122.215828 73.387)
-		(end 124.071528 73.387)
+		(start 118.16962 79.801141)
+		(end 118.16962 77.43038)
 		(width 0.2)
 		(layer "B.Cu")
@@
 	)
 	(segment
-		(start 125.434189 61.134189)
-		(end 118.2 53.9)
+		(start 122.215828 73.387)
+		(end 124.071528 73.387)
 		(width 0.2)
 		(layer "B.Cu")
@@
 	)
 	(segment
-		(start 111.607463 87.812537)
-		(end 110.8 88.62)
+		(start 125.434189 61.134189)
+		(end 118.2 53.9)
 		(width 0.2)
 		(layer "B.Cu")
@@
 	)
 	(segment
-		(start 111.607463 87.407463)
-		(end 118.16962 80.845305)
+		(start 117.39 80.580761)
+		(end 118.16962 79.801141)
 		(width 0.2)
 		(layer "B.Cu")
@@
 	)
 	(segment
-		(start 118.16962 77.43038)
-		(end 121.7 73.9)
+		(start 111.65 87.364925)
+		(end 117.39 81.624925)
 		(width 0.2)
 		(layer "B.Cu")
@@
 	)
 	(segment
+		(start 117.39 81.624925)
+		(end 117.39 80.580761)
+		(width 0.2)
+		(layer "B.Cu")
+		(net "/PA10")
+	)
+	(segment
 		(start 126.225 71.175811)
 		(end 125.434189 70.385)
@@
 	)
 	(segment
-		(start 118.16962 80.845305)
-		(end 118.16962 77.43038)
+		(start 110.8 88.62)
+		(end 111.65 87.77)
 		(width 0.2)
 		(layer "B.Cu")
@@
 	)
 	(segment
-		(start 118.2 53.9)
-		(end 118.2 52)
+		(start 111.65 87.77)
+		(end 111.65 87.364925)
+		(width 0.2)
+		(layer "B.Cu")
+		(net "/PA10")
+	)
+	(segment
+		(start 118.16962 77.43038)
+		(end 121.7 73.9)
 		(width 0.2)
 		(layer "B.Cu")
@@
 	)
 	(segment
-		(start 111.607463 87.407463)
-		(end 111.607463 87.812537)
+		(start 118.2 53.9)
+		(end 118.2 52)
 		(width 0.2)
 		(layer "B.Cu")

Commit message: Update stor.kicad_pcb
Routing:
- net /VBUS: track 48.9 -> 51.2 mm, vias 4 -> 7
Changed lines of the file:
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@@
-	)
-	(via
-		(at 124.025 46.93)
-		(size 0.6)
-		(drill 0.3)
-		(layers "F.Cu" "B.Cu")
-		(net "GND")
 	)
 	(via
@@
 		(drill 0.3)
 		(layers "F.Cu" "B.Cu")
+		(net "GND")
+	)
+	(via
+		(at 125.62 46.9)
+		(size 0.6)
+		(drill 0.3)
+		(layers "F.Cu" "B.Cu")
+		(free yes)
 		(net "GND")
 	)
@@
 	)
 	(segment
+		(start 116.5 37)
+		(end 116.5 38.9875)
+		(width 0.4)
+		(layer "F.Cu")
+		(net "/VBUS")
+	)
+	(segment
 		(start 125.58 42.167)
 		(end 125.58 42.430227)
@@
 	)
 	(segment
-		(start 116.2375 38.9875)
-		(end 115.5 38.25)
-		(width 0.2)
-		(layer "F.Cu")
-		(net "/VBUS")
-	)
-	(segment
 		(start 126.65 48.35)
 		(end 127.3 47.7)
@@
 	)
 	(segment
-		(start 116.5 38.9875)
+		(start 115.615 37.385)
+		(end 115.91 37.68)
+		(width 0.4)
+		(layer "F.Cu")
+		(net "/VBUS")
+	)
+	(segment
+		(start 116.115 37.385)
 		(end 116.5 37)
-		(width 0.2)
+		(width 0.4)
 		(layer "F.Cu")
 		(net "/VBUS")
@@
 	)
 	(segment
+		(start 115.5 38.25)
+		(end 115.7625 38.25)
+		(width 0.4)
+		(layer "F.Cu")
+		(net "/VBUS")
+	)
+	(segment
+		(start 115.91 37.68)
+		(end 115.94 37.68)
+		(width 0.4)
+		(layer "F.Cu")
+		(net "/VBUS")
+	)
+	(segment
+		(start 116.5 38.24)
+		(end 116.5 38.9875)
+		(width 0.4)
+		(layer "F.Cu")
+		(net "/VBUS")
+	)
+	(segment
 		(start 127.575 47.025)
 		(end 127.375 47.225)
@@
 	)
 	(segment
+		(start 115.615 37.385)
+		(end 116.115 37.385)
+		(width 0.4)
+		(layer "F.Cu")
+		(net "/VBUS")
+	)
+	(segment
 		(start 125.092951 42.917276)
 		(end 124.238205 42.917276)
@@
 	)
 	(segment
+		(start 115.615 37.385)
+		(end 115.615 38.135)
+		(width 0.4)
+		(layer "F.Cu")
+		(net "/VBUS")
+	)
+	(segment
+		(start 115.7625 38.25)
+		(end 116.5 38.9875)
+		(width 0.4)
+		(layer "F.Cu")
+		(net "/VBUS")
+	)
+	(segment
 		(start 127.3 47.439339)
 		(end 127.3 47.7)
@@
 	)
 	(segment
+		(start 115.615 38.135)
+		(end 115.5 38.25)
+		(width 0.4)
+		(layer "F.Cu")
+		(net "/VBUS")
+	)
+	(segment
 		(start 125.44 48.4125)
 		(end 125.55125 48.30125)
@@
 	)
 	(segment
+		(start 126.27 48.35)
+		(end 126.65 48.35)
+		(width 0.4)
+		(layer "F.Cu")
+		(net "/VBUS")
+	)
+	(segment
+		(start 115.94 37.68)
+		(end 116.5 38.24)
+		(width 0.4)
+		(layer "F.Cu")
+		(net "/VBUS")
+	)
+	(segment
 		(start 130.3 42.35)
 		(end 130.3 46.65)
@@
 	)
 	(segment
-		(start 125.718817 48.35)
-		(end 126.65 48.35)
-		(width 0.4)
-		(layer "F.Cu")
-		(net "/VBUS")
-	)
-	(segment
 		(start 127.375 47.085)
 		(end 127.14 46.85)
@@
 	)
 	(via
+		(at 115.615 37.385)
+		(size 0.6)
+		(drill 0.3)
+		(layers "F.Cu" "B.Cu")
+		(net "/VBUS")
+	)
+	(via
+		(at 126.27 48.35)
+		(size 0.6)
+		(drill 0.3)
+		(layers "F.Cu" "B.Cu")
+		(net "/VBUS")
+	)
+	(via
+		(at 125.289409 48.779409)
+		(size 0.6)
+		(drill 0.3)
+		(layers "F.Cu" "B.Cu")
+		(net "/VBUS")
+	)
+	(via
 		(at 115.5 38.25)
 		(size 0.6)
@@
 	)
 	(segment
+		(start 125.718817 48.35)
+		(end 126.27 48.35)
+		(width 0.4)
+		(layer "In2.Cu")
+		(net "/VBUS")
+	)
+	(segment
 		(start 122.1 49.35)
 		(end 124.718817 49.35)
@@
 	(segment
 		(start 124.718817 49.35)
-		(end 125.718817 48.35)
-		(width 0.4)
-		(layer "In2.Cu")
-		(net "/VBUS")
-	)
-	(segment
-		(start 115.5 38.25)
-		(end 115.5 37.5)
+		(end 125.289409 48.779409)
 		(width 0.4)
 		(layer "In2.Cu")
@@
 	)
 	(segment
-		(start 115.75 37.25)
-		(end 116.25 37.25)
-		(width 0.4)
-		(layer "In2.Cu")
-		(net "/VBUS")
-	)
-	(segment
-		(start 116.25 37.25)
-		(end 116.5 37)
-		(width 0.4)
-		(layer "In2.Cu")
-		(net "/VBUS")
-	)
-	(segment
-		(start 115.5 37.5)
-		(end 115.75 37.25)
-		(width 0.4)
-		(layer "In2.Cu")
-		(net "/VBUS")
-	)
-	(segment
 		(start 116.133959 43.949029)
 		(end 116.495911 44.310981)
 		(width 0.4)
 		(layer "In2.Cu")
+		(net "/VBUS")
+	)
+	(segment
+		(start 125.289409 48.779409)
+		(end 125.718817 48.35)
+		(width 0.4)
+		(layer "In2.Cu")

Commit message: yes
Parts:
- added kobee-studio-6A814325: Kobee Studio, kobee-studio-6A814325, B.Cu at (127.3, 71.7)
- added kobee-studio-6A814354: Kobee Studio, kobee-studio-6A814354, B.Cu at (125.7, 68.9)
- added kobee-studio-6A8143AA: Kobee Studio, kobee-studio-6A8143AA, B.Cu at (110.8, 81.1)
- added kobee-studio-6A8143BF: Kobee Studio, kobee-studio-6A8143BF, B.Cu at (112.5, 78.4)
- added kobee-studio-6A8144FF: Kobee Studio, kobee-studio-6A8144FF, F.Cu at (110.2, 76.2)
- added kobee-studio-6A81454B: Kobee Studio, kobee-studio-6A81454B, F.Cu at (129.8, 76.2)
- moved SW2 0.10 mm to (125.5, 76.2)
Other:
- board text removed: "BOOT0"
- board text removed: "CLK"
- board text removed: "GND"
- board text removed: "IO"
- board text removed: "NRST"
- board text removed: "RESET"
- board text removed: "RX"
- board text removed: "STM32H7 inside"
- board text removed: "SWD"
- board text removed: "TX"
- board text removed: "UART"
- board text removed: "USB2.0"
- board text removed: "VDD"
